File: CAN.kicad_sch (KiCad schematic)
At the start: 11 parts, among them J4 Conn_01x02, J6 Conn_01x02, U6 MCP2562FD-H/SN

Commit message: 回路図（ひとまず完成）
Parts:
- D14, D17: footprint (none) -> LED_THT:LED_D3.0mm
- R38: footprint (none) -> Resistor_SMD:R_0603_1608Metric_Pad0.98x0.95mm_HandSolder
- U6: footprint MCP2562FD-H/SN:SOIC8-N_MC_MCH -> MCP2652FD_H_SN:SOIC8-N_MC_MCH-L
Other:
- note added: "MCR03SEQPF1200"
Changed lines of the file:
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@@
 	(generator_version "10.0")
 	(paper "A4")
+	(text "MCR03SEQPF1200"
+		(exclude_from_sim no)
+		(at 208.28 100.584 0)
+		(effects
+			(font
+				(size 1.27 1.27)
+			)
+		)
+	)
 	(junction
 		(at 185.42 91.44)
@@
 			)
 		)
-		(property "Footprint" ""
+		(property "Footprint" "LED_THT:LED_D3.0mm"
 			(at 99.06 76.2 0)
 			(hide yes)
@@
 			)
 		)
-		(property "Footprint" ""
+		(property "Footprint" "LED_THT:LED_D3.0mm"
 			(at 107.95 76.2 0)
 			(hide yes)
@@
 			)
 		)
-		(property "Footprint" "MCP2562FD-H/SN:SOIC8-N_MC_MCH"
+		(property "Footprint" "MCP2652FD_H_SN:SOIC8-N_MC_MCH-L"
 			(at 113.03 86.36 0)
 			(hide yes)
@@
 			)
 		)
-		(property "Footprint" ""
+		(property "Footprint" "Resistor_SMD:R_0603_1608Metric_Pad0.98x0.95mm_HandSolder"
 			(at 196.85 107.188 90)
 			(hide yes)

Commit message: 抵抗器のフットプリントを策定
Parts:
- C12, C13: footprint (none) -> Capacitor_SMD:C_0603_1608Metric_Pad1.08x0.95mm_HandSolder
- R33, R34: footprint (none) -> Resistor_SMD:R_0603_1608Metric_Pad0.98x0.95mm_HandSolder
- R39: footprint (none) -> Resistor_SMD:R_0805_2012Metric_Pad1.20x1.40mm_HandSolder
Changed lines of the file:
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@@
 			)
 		)
-		(property "Footprint" ""
+		(property "Footprint" "Resistor_SMD:R_0805_2012Metric_Pad1.20x1.40mm_HandSolder"
 			(at 233.172 100.33 90)
 			(hide yes)
@@
 			)
 		)
-		(property "Footprint" ""
+		(property "Footprint" "Resistor_SMD:R_0603_1608Metric_Pad0.98x0.95mm_HandSolder"
 			(at 97.282 68.58 90)
 			(hide yes)
@@
 			)
 		)
-		(property "Footprint" ""
+		(property "Footprint" "Capacitor_SMD:C_0603_1608Metric_Pad1.08x0.95mm_HandSolder"
 			(at 75.8952 100.33 0)
 			(hide yes)
@@
 			)
 		)
-		(property "Footprint" ""
+		(property "Footprint" "Resistor_SMD:R_0603_1608Metric_Pad0.98x0.95mm_HandSolder"
 			(at 106.172 68.58 90)
 			(hide yes)
@@
 			)
 		)
-		(property "Footprint" ""
+		(property "Footprint" "Capacitor_SMD:C_0603_1608Metric_Pad1.08x0.95mm_HandSolder"
 			(at 176.2252 104.14 0)
 			(hide yes)
