File: MCU.kicad_sch (KiCad schematic)
At the start: 23 parts, among them J5 Conn_01x05, SW3 SW_SPDT, SW4 SW_Push, U7 STM32H503CBTx, X1 MU00525-32.768K

Commit message: 回路図（ひとまず完成）
Parts:
- J5: footprint (none) -> Connector_PinHeader_2.54mm:PinHeader_1x05_P2.54mm_Vertical
Connections:
- net GPIO_1: now reaches U7.13 (PA3)
- net GPIO_2: now reaches U7.14 (PA4)
- net GPIO_3: now reaches U7.15 (PA5)
- net GPIO_4: now reaches U7.16 (PA6)
- net GPIO_5: now reaches U7.17 (PA7)
- net GPIO_６: now reaches U7.18 (PB0)
- net GPIO_7: now reaches U7.19 (PB1)
- net GPIO_8: now reaches U7.20 (PB2)
- net GPIO_9: now reaches U7.21 (PB10)
- net GPIO_LM_1: now reaches U7.27 (PB14)
- net GPIO_LM_2: now reaches U7.28 (PB15)
- net GPIO_LM_3: now reaches U7.29 (PA8)
- net GPIO_LM_4: now reaches U7.30 (PA9)
- net GPIO_LM_5: now reaches U7.31 (PA10)
- net GPIO_LM_6: now reaches U7.32 (PA11)
- net GPIO_LM_7: now reaches U7.33 (PA12)
- no-connect marks 22 -> 8

Commit message: 抵抗器のフットプリントを策定
Parts:
- C28, C30, C31, C34, C35, C36, C37, C38, C40, C41, C42, C43, C44, C45: footprint (none) -> Capacitor_SMD:C_0603_1608Metric_Pad1.08x0.95mm_HandSolder
- R35, R40: footprint (none) -> Resistor_SMD:R_0603_1608Metric_Pad0.98x0.95mm_HandSolder
- SW3: footprint (none) -> Connector_PinHeader_2.54mm:PinHeader_1x03_P2.54mm_Vertical
- SW4: footprint (none) -> Button_Switch_THT:SW_PUSH-12mm
