File: MCU.kicad_sch (KiCad schematic)
At the start: 23 parts, among them J5 Conn_01x05, SW3 SW_SPDT, SW4 SW_Push, U7 STM32H503CBTx, X1 MU00525-32.768K

Commit message: サーボ電源と通信線一部
Parts:
- added R2, R3: 33, Resistor_SMD:R_0603_1608Metric_Pad0.98x0.95mm_HandSolder, symbol Device:R
Connections:
- net PA13-JTMS-SWDIO: now also R3.2; no longer J5.4 (Pin_4)
- net PA14-JTCK-SWCLK: now also R2.1; no longer J5.2 (Pin_2)
- net GPIO_６ renamed GPIO_6
- new net: J5.4 (Pin_4), R3.1
- new net: J5.2 (Pin_2), R2.2

Commit message: DRCのエラー・警告を一部無視したけど問題ないよね
Parts:
- C31, C34, C36, C37, C38, C41: LCSC (none) -> C1591

Commit message: 一部修正、製造ファイル出力
Parts:
- C31, C34, C36, C37, C38, C41: LCSC C1591 -> (none)
- SW3: footprint Connector_PinHeader_2.54mm:PinHeader_1x03_P2.54mm_Vertical -> SlideSW:SlideSW
