File: CMFD-LMSE.kicad_pcb (KiCad board)
At the start: 2 copper layers, 130 parts, among them J1 Conn_01x02, J10 Conn_01x02, J11 Conn_01x02, J12 Conn_01x02, J2 Conn_01x02, J3 ZX62-B-5PA_33_, J4 Conn_01x02, J5 Conn_01x05, J6 Conn_01x02, J7 Conn_01x02, J8 Conn_01x02, J9 Conn_01x02, SW3 SW_SPDT, SW4 SW_Push, U1 MPM3610GQV-Z, U2 CH340E, U4 TPS2117DRLR, U5 BD33IC0WEFJ-E2, U6 MCP2562FD-H/SN, U7 STM32H503CBTx, X1 MU00525-32.768K

Commit message: クラッシュ直後
Parts:
- GPIO1, GPIO2, GPIO3, GPIO4, GPIO5, GPIO6, GPIO7, GPIO8, GPIO9: footprint Connector_JST:JST_XA_S03B-XASK-1_1x03_P2.50mm_Horizontal -> DF1B_3P_2_5DSA:CONN3_DF1B-3P_HIR
- R26, R28: footprint KIR03EZPF1003:RES_R0603_ROM-M -> KIR03EZPF1003:RES_R0603_ROM-L
- TP1, TP2, TP3, TP4: footprint TestPoint:TestPoint_Pad_3.0x3.0mm -> TestPoint:TestPoint_Pad_1.5x1.5mm
- moved GPIO7 242.9 mm to (184.2, 123.9)
- moved H4 238.1 mm to (189.5, 136.5)
- moved D5 235.6 mm to (190.3, 119.0), turned to 180 degrees
- moved GPIO4 229.8 mm to (148.7, 124.0)
- moved GPIO5 229.7 mm to (160.4, 124.0)
- moved GPIO6 229.5 mm to (172.2, 124.0)
- moved D6 226.6 mm to (178.6, 119.0), turned to 180 degrees
- moved GPIO8 226.1 mm to (185.9, 110.3), turned to 90 degrees
- moved R16 224.4 mm to (186.6, 119.0), turned to 180 degrees
- moved R12 223.3 mm to (180.7, 111.6), turned to -90 degrees
- moved GPIO1 222.6 mm to (113.2, 124.0)
- moved GPIO2 222.5 mm to (125.1, 124.1)
- moved GPIO3 222.4 mm to (136.9, 124.0)
- moved R11 220.7 mm to (182.8, 119.0), turned to 180 degrees
- moved D4 220.0 mm to (180.7, 104.0), turned to -90 degrees
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Connections:
- net Net-(IN1-Pin_2) renamed +BATT
- R14 pad 1: Net-(GPIO9-Pin_1) -> Net-(D3-A)
- R14 pad 2: Net-(D3-A) -> Net-(GPIO9-Pin_1)
- R15 pad 1: Net-(GPIO8-Pin_1) -> Net-(D4-A)
- R15 pad 2: Net-(D4-A) -> Net-(GPIO8-Pin_1)
- R16 pad 1: Net-(GPIO7-Pin_1) -> Net-(D5-A)
- R16 pad 2: Net-(D5-A) -> Net-(GPIO7-Pin_1)
- R17 pad 1: Net-(GPIO6-Pin_1) -> Net-(D6-A)
- R17 pad 2: Net-(D6-A) -> Net-(GPIO6-Pin_1)
- R18 pad 1: Net-(GPIO5-Pin_1) -> Net-(D7-A)
- R18 pad 2: Net-(D7-A) -> Net-(GPIO5-Pin_1)
- R19 pad 1: Net-(GPIO4-Pin_1) -> Net-(D8-A)
- R19 pad 2: Net-(D8-A) -> Net-(GPIO4-Pin_1)
- R20 pad 1: Net-(GPIO3-Pin_1) -> Net-(D9-A)
- R20 pad 2: Net-(D9-A) -> Net-(GPIO3-Pin_1)
- R21 pad 1: Net-(GPIO2-Pin_1) -> Net-(D10-A)
- R21 pad 2: Net-(D10-A) -> Net-(GPIO2-Pin_1)
- R22 pad 1: Net-(GPIO1-Pin_1) -> Net-(D11-A)
- R22 pad 2: Net-(D11-A) -> Net-(GPIO1-Pin_1)
Routing:
- net VIN: track 0.00 -> 28.9 mm
- net GND: track 0.00 -> 12.7 mm, vias 0 -> 6
- net Net-(F2-Pad1): track 0.00 -> 10.7 mm
- net Net-(D13-ANODE): track 0.00 -> 9.60 mm
- net Net-(GPIO3-Pin_2): track 0.00 -> 4.50 mm
- net Net-(GPIO1-Pin_2): track 0.00 -> 4.45 mm
- net Net-(GPIO8-Pin_2): track 0.00 -> 4.30 mm
- net Net-(GPIO6-Pin_2): track 0.00 -> 4.20 mm
- net Net-(GPIO5-Pin_2): track 0.00 -> 4.20 mm
- net Net-(GPIO2-Pin_2): track 0.00 -> 4.05 mm
- net Net-(GPIO7-Pin_2): track 0.00 -> 4.05 mm
- net Net-(GPIO4-Pin_2): track 0.00 -> 4.00 mm
- net Net-(U1-EN): track 0.00 -> 3.91 mm
- net Net-(D12-A): track 0.00 -> 2.30 mm
- net Net-(U1-AAM): track 0.00 -> 1.85 mm
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- added copper zone on In1.Cu, net +BATT
- added copper zone on In1.Cu, net /PowerAndUSB/VIN+
Other:
- board outline added: 100 x 80 mm
- copper layers 2 -> 4
- board text added: "H"
- board text added: "L"
- board text added: "Power"

Commit message: U2とU4にカスタムルールを設定
Parts:
- moved R1 0.60 mm to (121.0, 111.5)
Routing:
- net Net-(U1-FB): track 0.00 -> 7.27 mm, vias 0 -> 3
- net /PowerAndUSB/VIN_5V: track 1.06 -> 6.70 mm
- net GND: track 12.7 -> 17.7 mm, vias 6 -> 8
- net /PowerAndUSB/VIN+: track 0.00 -> 2.42 mm, vias 1 -> 2
- net Net-(U1-AAM): track 1.85 -> 0.29 mm
- net VIN: track 28.9 -> 27.4 mm
- net Net-(U1-EN): track 3.91 -> 5.02 mm, vias 0 -> 2
