File: CMFD-LMSE.kicad_sch (KiCad schematic)
At the start: 59 parts, among them J1 Conn_01x02, J10 Conn_01x02, J11 Conn_01x02, J12 Conn_01x02, J7 Conn_01x02, J8 Conn_01x02, J9 Conn_01x02

Commit message: クラッシュ直後
Parts:
- GPIO1, GPIO2, GPIO3, GPIO4, GPIO5, GPIO6, GPIO7, GPIO8, GPIO9: footprint Connector_JST:JST_XA_S03B-XASK-1_1x03_P2.50mm_Horizontal -> DF1B_3P_2_5DSA:CONN3_DF1B-3P_HIR
Connections:
- net +BATT: now reaches IN1.2 (Pin_2), JP1.1 (A), JP2.1 (A), JP3.1 (A), JP4.1 (A), JP5.1 (A), JP6.1 (A), JP7.1 (A), JP8.1 (A), JP9.1 (A), R23.1
- net at GPIO3.1 (Pin_1), R7.2: now also R20.2; no longer R20.1
- net at D9.2 (A): now also R20.1; no longer R20.2
- net at GPIO4.1 (Pin_1), R8.2: now also R19.2; no longer R19.1
- net at GPIO6.1 (Pin_1), R10.2: now also R17.2; no longer R17.1
- net at D6.2 (A): now also R17.1; no longer R17.2
- net at GPIO7.1 (Pin_1), R11.2: now also R16.2; no longer R16.1
- net at D5.2 (A): now also R16.1; no longer R16.2
- net at GPIO8.1 (Pin_1), R12.2: now also R15.2; no longer R15.1
- net at D4.2 (A): now also R15.1; no longer R15.2
- net at GPIO9.1 (Pin_1), R13.2: now also R14.2; no longer R14.1
- net at D3.2 (A): now also R14.1; no longer R14.2
- net at GPIO5.1 (Pin_1), R9.2: now also R18.2; no longer R18.1
- net at D11.2 (A): now also R22.1; no longer R22.2
- net at D8.2 (A): now also R19.1; no longer R19.2
- net at GPIO1.1 (Pin_1), R5.2: now also R22.2; no longer R22.1
- net at D7.2 (A): now also R18.1; no longer R18.2
- net at GPIO2.1 (Pin_1), R6.2: now also R21.2; no longer R21.1
- net at D10.2 (A): now also R21.1; no longer R21.2
Other:
- moved on the sheet: D5, R14, R15, R16, R17, R18, R19, R20, R21, R22
Changed lines of the file:
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@@
 	)
 	(junction
+		(at 208.28 29.21)
+		(diameter 0)
+		(color 0 0 0 0)
+	)
+	(junction
 		(at 218.44 100.33)
 		(diameter 0)
@@
 	(wire
 		(pts
+			(xy 208.28 26.67) (xy 208.28 29.21)
+		)
+		(stroke
+			(width 0)
+			(type default)
+		)
+	)
+	(wire
+		(pts
 			(xy 152.4 52.07) (xy 201.93 52.07)
 		)
@@
 	(symbol
 		(lib_id "Device:R")
-		(at 190.5 124.46 0)
+		(at 190.5 124.46 180)
 		(unit 1)
 		(body_style 1)
@@
 		(dnp no)
 		(property "Reference" "R20"
-			(at 191.77 123.825 0)
+			(at 189.23 125.095 0)
 			(show_name no)
 			(do_not_autoplace no)
@@
 		)
 		(property "Value" "1K"
-			(at 191.77 126.365 0)
+			(at 189.23 122.555 0)
 			(show_name no)
 			(do_not_autoplace no)
@@
 		)
 		(property "Footprint" "Resistor_SMD:R_0603_1608Metric_Pad0.98x0.95mm_HandSolder"
-			(at 188.722 124.46 90)
+			(at 192.278 124.46 90)
 			(hide yes)
 			(show_name no)
@@
 	)
 	(symbol
+		(lib_id "power:+BATT")
+		(at 208.28 26.67 0)
+		(unit 1)
+		(body_style 1)
+		(exclude_from_sim no)
+		(in_bom yes)
+		(on_board yes)
+		(in_pos_files yes)
+		(dnp no)
+		(fields_autoplaced yes)
+		(property "Reference" "#PWR022"
+			(at 208.28 30.48 0)
+			(hide yes)
+			(show_name no)
+			(do_not_autoplace no)
+			(effects
+				(font
+					(size 1.27 1.27)
+				)
+			)
+		)
+		(property "Value" "+BATT"
+			(at 208.28 21.59 0)
+			(show_name no)
+			(do_not_autoplace no)
+			(effects
+				(font
+					(size 1.27 1.27)
+				)
+			)
+		)
+		(property "Footprint" ""
+			(at 208.28 26.67 0)
+			(hide yes)
+			(show_name no)
+			(do_not_autoplace no)
+			(effects
+				(font
+					(size 1.27 1.27)
+				)
+			)
+		)
+		(property "Datasheet" ""
+			(at 208.28 26.67 0)
+			(hide yes)
+			(show_name no)
+			(do_not_autoplace no)
+			(effects
+				(font
+					(size 1.27 1.27)
+				)
+			)
+		)
+		(property "Description" "Power symbol creates a global label with name \"+BATT\""
+			(at 208.28 26.67 0)
+			(hide yes)
+			(show_name no)
+			(do_not_autoplace no)
+			(effects
+				(font
+					(size 1.27 1.27)
+				)
+			)
+		)
+		(pin "1"
+		)
+		(instances
+			(project "CMFD-LMSE"
+				(path "/1c8cd19f-66ef-4296-985a-c19890cd74b7"
+					(reference "#PWR022")
+					(unit 1)
+				)
+			)
+		)
+	)
+	(symbol
 		(lib_id "Jumper:SolderJumper_3_Open")
 		(at 213.36 100.33 0)
@@
 			)
 		)
-		(property "Footprint" "Connector_JST:JST_XA_S03B-XASK-1_1x03_P2.50mm_Horizontal"
+		(property "Footprint" "DF1B_3P_2_5DSA:CONN3_DF1B-3P_HIR"
 			(at 238.76 71.12 0)
 			(hide yes)
@@
 			)
 		)
-		(property "Footprint" "Connector_JST:JST_XA_S03B-XASK-1_1x03_P2.50mm_Horizontal"
+		(property "Footprint" "DF1B_3P_2_5DSA:CONN3_DF1B-3P_HIR"
 			(at 238.76 78.74 0)
 			(hide yes)
@@
 	(symbol
 		(lib_id "Device:R")
-		(at 172.72 124.46 0)
+		(at 172.72 124.46 180)
 		(unit 1)
 		(body_style 1)
@@
 		(dnp no)
 		(property "Reference" "R17"
-			(at 173.99 123.825 0)
+			(at 171.45 125.095 0)
 			(show_name no)
 			(do_not_autoplace no)
@@
 		)
 		(property "Value" "1K"
-			(at 173.99 126.365 0)
+			(at 171.45 122.555 0)
 			(show_name no)
 			(do_not_autoplace no)
@@
 		)
 		(property "Footprint" "Resistor_SMD:R_0603_1608Metric_Pad0.98x0.95mm_HandSolder"
-			(at 170.942 124.46 90)
+			(at 174.498 124.46 90)
 			(hide yes)
 			(show_name no)
@@
 	(symbol
 		(lib_id "Device:R")
-		(at 167.64 124.46 0)
+		(at 167.64 124.46 180)
 		(unit 1)
 		(body_style 1)
@@
 		(dnp no)
 		(property "Reference" "R16"
-			(at 168.91 123.825 0)
+			(at 166.37 125.095 0)
 			(show_name no)
 			(do_not_autoplace no)
@@
 		)
 		(property "Value" "1K"
-			(at 168.91 126.365 0)
+			(at 166.37 122.555 0)
 			(show_name no)
 			(do_not_autoplace no)
@@
 		)
 		(property "Footprint" "Resistor_SMD:R_0603_1608Metric_Pad0.98x0.95mm_HandSolder"
-			(at 165.862 124.46 90)
+			(at 169.418 124.46 90)
 			(hide yes)
 			(show_name no)
@@
 	(symbol
 		(lib_id "Device:R")
-		(at 161.29 124.46 0)
+		(at 161.29 124.46 180)
 		(unit 1)
 		(body_style 1)
@@
 		(dnp no)
 		(property "Reference" "R15"
-			(at 162.56 123.825 0)
+			(at 160.02 125.095 0)
 			(show_name no)
 			(do_not_autoplace no)
@@
 		)
 		(property "Value" "1K"
-			(at 162.56 126.365 0)
+			(at 160.02 122.555 0)
 			(show_name no)
 			(do_not_autoplace no)
@@
 		)
 		(property "Footprint" "Resistor_SMD:R_0603_1608Metric_Pad0.98x0.95mm_HandSolder"
-			(at 159.512 124.46 90)
+			(at 163.068 124.46 90)
 			(hide yes)
 			(show_name no)
@@
 	(symbol
 		(lib_id "Device:R")
-		(at 156.21 124.46 0)
+		(at 156.21 124.46 180)
 		(unit 1)
 		(body_style 1)
@@
 		(dnp no)
 		(property "Reference" "R14"
-			(at 157.48 123.825 0)
+			(at 154.94 125.095 0)
 			(show_name no)
 			(do_not_autoplace no)
@@
 		)
 		(property "Value" "1K"
-			(at 157.48 126.365 0)
+			(at 154.94 122.555 0)
 			(show_name no)
 			(do_not_autoplace no)
@@
 		)
 		(property "Footprint" "Resistor_SMD:R_0603_1608Metric_Pad0.98x0.95mm_HandSolder"
-			(at 154.432 124.46 90)
+			(at 157.988 124.46 90)
 			(hide yes)
 			(show_name no)
@@
 			)
 		)
-		(property "Footprint" "Connector_JST:JST_XA_S03B-XASK-1_1x03_P2.50mm_Horizontal"
+		(property "Footprint" "DF1B_3P_2_5DSA:CONN3_DF1B-3P_HIR"
 			(at 238.76 111.76 0)
 			(hide yes)
@@
 			)
 		)
-		(property "Footprint" "Connector_JST:JST_XA_S03B-XASK-1_1x03_P2.50mm_Horizontal"
+		(property "Footprint" "DF1B_3P_2_5DSA:CONN3_DF1B-3P_HIR"
 			(at 238.76 87.63 0)
 			(hide yes)
@@
 		(lib_name "LED_1")
 		(lib_id "Device:LED")
-		(at 167.64 132.08 90)
+		(at 167.64 132.08 270)
+		(mirror x)
 		(unit 1)
 		(body_style 1)
@@
 		(dnp no)
 		(property "Reference" "D5"
-			(at 168.91 129.54 90)
+			(at 166.37 129.54 90)
 			(show_name no)
 			(do_not_autoplace no)
@@
 		)
 		(property "Value" "LED"
-			(at 170.815 130.81 0)
+			(at 164.465 130.81 0)
 			(show_name no)
 			(do_not_autoplace no)
@@
 			)
 		)
-		(property "Footprint" "Connector_JST:JST_XA_S03B-XASK-1_1x03_P2.50mm_Horizontal"
+		(property "Footprint" "DF1B_3P_2_5DSA:CONN3_DF1B-3P_HIR"
 			(at 238.76 120.65 0)
 			(hide yes)
@@
 	(symbol
 		(lib_id "Device:R")
-		(at 201.93 124.46 0)
+		(at 201.93 124.46 180)
 		(unit 1)
 		(body_style 1)
@@
 		(dnp no)
 		(property "Reference" "R22"
-			(at 203.2 123.825 0)
+			(at 200.66 125.095 0)
 			(show_name no)
 			(do_not_autoplace no)
@@
 		)
 		(property "Value" "1K"
-			(at 203.2 126.365 0)
+			(at 200.66 122.555 0)
 			(show_name no)
 			(do_not_autoplace no)
@@
 		)
 		(property "Footprint" "Resistor_SMD:R_0603_1608Metric_Pad0.98x0.95mm_HandSolder"
-			(at 200.152 124.46 90)
+			(at 203.708 124.46 90)
 			(hide yes)
 			(show_name no)
@@
 	(symbol
 		(lib_id "Device:R")
-		(at 179.07 124.46 0)
+		(at 179.07 124.46 180)
 		(unit 1)
 		(body_style 1)
@@
 		(dnp no)
 		(property "Reference" "R18"
-			(at 180.34 123.825 0)
+			(at 177.8 125.095 0)
 			(show_name no)
 			(do_not_autoplace no)
@@
 		)
 		(property "Value" "1K"
-			(at 180.34 126.365 0)
+			(at 177.8 122.555 0)
 			(show_name no)
 			(do_not_autoplace no)
@@
 		)
 		(property "Footprint" "Resistor_SMD:R_0603_1608Metric_Pad0.98x0.95mm_HandSolder"
-			(at 177.292 124.46 90)
+			(at 180.848 124.46 90)
 			(hide yes)
 			(show_name no)
@@
 			)
 		)
-		(property "Footprint" "Connector_JST:JST_XA_S03B-XASK-1_1x03_P2.50mm_Horizontal"
+		(property "Footprint" "DF1B_3P_2_5DSA:CONN3_DF1B-3P_HIR"
 			(at 238.76 54.61 0)
 			(hide yes)
@@
 			)
 		)
-		(property "Footprint" "Connector_JST:JST_XA_S03B-XASK-1_1x03_P2.50mm_Horizontal"
+		(property "Footprint" "DF1B_3P_2_5DSA:CONN3_DF1B-3P_HIR"
 			(at 238.76 104.14 0)
 			(hide yes)
@@
 	(symbol
 		(lib_id "Device:R")
-		(at 184.15 124.46 0)
+		(at 184.15 124.46 180)
 		(unit 1)
 		(body_style 1)
@@
 		(dnp no)
 		(property "Reference" "R19"
-			(at 185.42 123.825 0)
+			(at 182.88 125.095 0)
 			(show_name no)
 			(do_not_autoplace no)
@@
 		)
 		(property "Value" "1K"
-			(at 185.42 126.365 0)
+			(at 182.88 122.555 0)
 			(show_name no)
 			(do_not_autoplace no)
@@
 		)
 		(property "Footprint" "Resistor_SMD:R_0603_1608Metric_Pad0.98x0.95mm_HandSolder"
-			(at 182.372 124.46 90)
+			(at 185.928 124.46 90)
 			(hide yes)
 			(show_name no)
@@
 			)
 		)
-		(property "Footprint" "Connector_JST:JST_XA_S03B-XASK-1_1x03_P2.50mm_Horizontal"
+		(property "Footprint" "DF1B_3P_2_5DSA:CONN3_DF1B-3P_HIR"
 			(at 238.76 62.23 0)
 			(hide yes)
@@
 	(symbol
 		(lib_id "Device:R")
-		(at 195.58 124.46 0)
+		(at 195.58 124.46 180)
 		(unit 1)
 		(body_style 1)
@@
 		(dnp no)
 		(property "Reference" "R21"
-			(at 196.85 123.825 0)
+			(at 194.31 125.095 0)
 			(show_name no)
 			(do_not_autoplace no)
@@
 		)
 		(property "Value" "1K"
-			(at 196.85 126.365 0)
+			(at 194.31 122.555 0)
 			(show_name no)
 			(do_not_autoplace no)
@@
 		)
 		(property "Footprint" "Resistor_SMD:R_0603_1608Metric_Pad0.98x0.95mm_HandSolder"
-			(at 193.802 124.46 90)
+			(at 197.358 124.46 90)
 			(hide yes)
 			(show_name no)
@@
 			)
 		)
-		(property "Footprint" "Connector_JST:JST_XA_S03B-XASK-1_1x03_P2.50mm_Horizontal"
+		(property "Footprint" "DF1B_3P_2_5DSA:CONN3_DF1B-3P_HIR"
 			(at 238.76 95.25 0)
 			(hide yes)

Commit message: サーボ電源と通信線一部
Connections:
- net MCU/GPIO_６ renamed MCU/GPIO_6
Other:
- sheet MCU ports: added GPIO_6; removed GPIO_６
Changed lines of the file:
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@@
 			)
 		)
-		(pin "GPIO_６" bidirectional
+		(pin "GPIO_6" bidirectional
 			(at 139.7 92.71 0)
 			(effects

Commit message: DRCのエラー・警告を一部無視したけど問題ないよね
Connections:
- net GND: no longer H1.1, H2.1, H3.1, H4.1
- no-connect marks 0 -> 4
