File: Power.kicad_sch (KiCad schematic)
At the start: 37 parts, among them J2 Conn_01x02, J3 ZX62-B-5PA_33_, U1 MPM3610GQV-Z, U2 CH340E, U4 TPS2117DRLR, U5 BD33IC0WEFJ-E2

Commit message: クラッシュ直後
Parts:
- R26, R28: footprint KIR03EZPF1003:RES_R0603_ROM-M -> KIR03EZPF1003:RES_R0603_ROM-L
- TP1, TP2, TP3, TP4: footprint TestPoint:TestPoint_Pad_3.0x3.0mm -> TestPoint:TestPoint_Pad_1.5x1.5mm
Changed lines of the file:
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@@
 			)
 		)
-		(property "Footprint" "KIR03EZPF1003:RES_R0603_ROM-M"
+		(property "Footprint" "KIR03EZPF1003:RES_R0603_ROM-L"
 			(at 146.558 140.97 90)
 			(hide yes)
@@
 			)
 		)
-		(property "Footprint" "TestPoint:TestPoint_Pad_3.0x3.0mm"
+		(property "Footprint" "TestPoint:TestPoint_Pad_1.5x1.5mm"
 			(at 231.14 43.18 0)
 			(hide yes)
@@
 			)
 		)
-		(property "Footprint" "TestPoint:TestPoint_Pad_3.0x3.0mm"
+		(property "Footprint" "TestPoint:TestPoint_Pad_1.5x1.5mm"
 			(at 274.32 55.88 0)
 			(hide yes)
@@
 			)
 		)
-		(property "Footprint" "KIR03EZPF1003:RES_R0603_ROM-M"
+		(property "Footprint" "KIR03EZPF1003:RES_R0603_ROM-L"
 			(at 56.388 152.4 90)
 			(hide yes)
@@
 			)
 		)
-		(property "Footprint" "TestPoint:TestPoint_Pad_3.0x3.0mm"
+		(property "Footprint" "TestPoint:TestPoint_Pad_1.5x1.5mm"
 			(at 391.16 76.2 0)
 			(hide yes)
@@
 			)
 		)
-		(property "Footprint" "TestPoint:TestPoint_Pad_3.0x3.0mm"
+		(property "Footprint" "TestPoint:TestPoint_Pad_1.5x1.5mm"
 			(at 237.49 52.07 0)
 			(hide yes)

Commit message: DRCのエラー・警告を一部無視したけど問題ないよね
Parts:
- C1, C6, C7, C9: LCSC (none) -> C5672
- C2, C5, C8: LCSC (none) -> C1591
- C4: footprint Capacitor_SMD:C_1206_3216Metric_Pad1.33x1.80mm_HandSolder -> Capacitor_THT:CP_Radial_D5.0mm_P2.50mm

Commit message: 一部修正、製造ファイル出力
Parts:
- C1, C6, C7, C9: LCSC C5672 -> (none)
- C2, C5, C8: LCSC C1591 -> (none)
Changed lines of the file:
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@@
 			)
 		)
-		(property "LCSC" "C1591"
+		(property "LCSC" ""
 			(at 203.2 156.21 0)
 			(hide yes)
@@
 			)
 		)
-		(property "LCSC" "C1591"
+		(property "LCSC" ""
 			(at 156.21 140.97 0)
 			(hide yes)
@@
 			)
 		)
-		(property "LCSC" "C5672"
+		(property "LCSC" ""
 			(at 168.91 140.97 0)
 			(hide yes)
@@
 			)
 		)
-		(property "LCSC" "C5672"
+		(property "LCSC" ""
 			(at 261.62 39.37 0)
 			(hide yes)
@@
 			)
 		)
-		(property "LCSC" "C1591"
+		(property "LCSC" ""
 			(at 33.02 149.86 0)
 			(hide yes)
@@
 			)
 		)
-		(property "LCSC" "C5672"
+		(property "LCSC" ""
 			(at 275.59 39.37 0)
 			(hide yes)
@@
 			)
 		)
-		(property "LCSC" "C5672"
+		(property "LCSC" ""
 			(at 26.67 162.56 0)
 			(hide yes)
